File: hardware/kicad/scoopy/scoopy.kicad_pcb (KiCad board)
At the start: 2 copper layers, 28 x 28 mm, 13 parts, among them J1 ESP32_SuperMini, J2 LD2410C, J3 Conn_01x04_Pin, SW1 SW_Push, SW2 SW_Push

Commit message: 1k Res was too bright for LEDs. Changed to 2.2k
Parts:
- R1, R2, R3: value 1k -> 2.2k
Other:
- board text added: "NHT"
- board text removed: "ZJVC"
Changed lines of the file:
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@@
 			)
 		)
-		(property "Value" "1k"
+		(property "Value" "2.2k"
 			(at 0 1.43 90)
 			(layer "F.Fab")
@@
 			)
 		)
-		(property "Datasheet" "https://www.farnell.com/datasheets/3693949.pdf"
+		(property "Datasheet" "https://4donline.ihs.com/images/VipMasterIC/IC/SCMP/SCMP-S-A0009547702/SCMP-S-A0009547702-1.pdf?hkey=6D3A4C79FDBF58556ACFDE234799DDF0"
 			(at 0 0 90)
 			(layer "F.Fab")
@@
 			)
 		)
-		(property "Supplier_PN" "2008335"
+		(property "Supplier_PN" "MCWR06X2201FTL"
 			(at 0 0 270)
 			(unlocked yes)
@@
 			)
 		)
-		(property "Link" "https://uk.farnell.com/bourns/cr0603-fx-1001elf/res-1k-1-0-1w-0603-thick-film/dp/2008335"
+		(property "Link" "https://uk.farnell.com/multicomp-pro/mcwr06x2201ftl/res-2k2-1-0-1w-0603-thick-film/dp/2447320"
 			(at 0 0 270)
 			(unlocked yes)
@@
 			)
 		)
-		(property "Value" "1k"
+		(property "Value" "2.2k"
 			(at 0 1.43 0)
 			(layer "F.Fab")
@@
 			)
 		)
-		(property "Datasheet" "https://www.farnell.com/datasheets/3693949.pdf"
+		(property "Datasheet" "https://4donline.ihs.com/images/VipMasterIC/IC/SCMP/SCMP-S-A0009547702/SCMP-S-A0009547702-1.pdf?hkey=6D3A4C79FDBF58556ACFDE234799DDF0"
 			(at 0 0 0)
 			(layer "F.Fab")
@@
 			)
 		)
-		(property "Supplier_PN" "2008335"
+		(property "Supplier_PN" "MCWR06X2201FTL"
 			(at 0 0 180)
 			(unlocked yes)
@@
 			)
 		)
-		(property "Link" "https://uk.farnell.com/bourns/cr0603-fx-1001elf/res-1k-1-0-1w-0603-thick-film/dp/2008335"
+		(property "Link" "https://uk.farnell.com/multicomp-pro/mcwr06x2201ftl/res-2k2-1-0-1w-0603-thick-film/dp/2447320"
 			(at 0 0 180)
 			(unlocked yes)
@@
 			)
 		)
-		(property "Value" "1k"
+		(property "Value" "2.2k"
 			(at 0 1.43 90)
 			(layer "F.Fab")
@@
 			)
 		)
-		(property "Datasheet" "https://www.farnell.com/datasheets/3693949.pdf"
+		(property "Datasheet" "https://4donline.ihs.com/images/VipMasterIC/IC/SCMP/SCMP-S-A0009547702/SCMP-S-A0009547702-1.pdf?hkey=6D3A4C79FDBF58556ACFDE234799DDF0"
 			(at 0 0 90)
 			(layer "F.Fab")
@@
 			)
 		)
-		(property "Supplier_PN" "2008335"
+		(property "Supplier_PN" "MCWR06X2201FTL"
 			(at 0 0 270)
 			(unlocked yes)
@@
 			)
 		)
-		(property "Link" "https://uk.farnell.com/bourns/cr0603-fx-1001elf/res-1k-1-0-1w-0603-thick-film/dp/2008335"
+		(property "Link" "https://uk.farnell.com/multicomp-pro/mcwr06x2201ftl/res-2k2-1-0-1w-0603-thick-film/dp/2447320"
 			(at 0 0 270)
 			(unlocked yes)
@@
 		)
 	)
-	(gr_text "ZJVC"
+	(gr_text "NHT"
 		(at 119 123.5 0)
 		(layer "F.SilkS")
@@
 			(justify left bottom)
 		)
-		(render_cache "ZJVC" 0
+		(render_cache "NHT" 0
 			(polygon
 				(pts
-					(xy 120.832065 123.16) (xy 119.122976 123.16) (xy 119.122976 122.784842) (xy 120.136706 121.518688)
-					(xy 119.172191 121.518688) (xy 119.172191 121.127899) (xy 120.777477 121.127899) (xy 120.777477 121.510872)
-					(xy 119.76509 122.769211) (xy 120.832065 122.769211)
+					(xy 121.109525 123.16) (xy 120.603942 123.16) (xy 119.740544 121.765251) (xy 119.740544 123.16)
+					(xy 119.25963 123.16) (xy 119.25963 121.127899) (xy 119.886723 121.127899) (xy 120.628611 122.292083)
+					(xy 120.628611 121.127899) (xy 121.109525 121.127899)
 				)
 			)
 			(polygon
 				(pts
-					(xy 122.256123 122.568932) (xy 122.243985 122.699788) (xy 122.208251 122.82038) (xy 122.148706 122.928624)
-					(xy 122.066224 123.018217) (xy 121.957963 123.093817) (xy 121.825767 123.151817) (xy 121.67601 123.186193)
-					(xy 121.477355 123.199078) (xy 121.212351 123.18882) (xy 120.993754 123.159389) (xy 120.993754 122.745764)
-					(xy 121.042969 122.745764) (xy 121.179501 122.793879) (xy 121.255725 122.80995) (xy 121.361217 122.816106)
-					(xy 121.495507 122.805076) (xy 121.581891 122.777393) (xy 121.648837 122.730274) (xy 121.691922 122.669682)
-					(xy 121.716297 122.599383) (xy 121.727337 122.521182) (xy 121.731489 122.314553) (xy 121.731489 121.49524)
-					(xy 121.265596 121.49524) (xy 121.265596 121.127899) (xy 122.256123 121.127899)
+					(xy 123.453646 123.16) (xy 122.929012 123.16) (xy 122.929012 122.261186) (xy 122.154396 122.261186)
+					(xy 122.154396 123.16) (xy 121.629762 123.16) (xy 121.629762 121.127899) (xy 122.154396 121.127899)
+					(xy 122.154396 121.870397) (xy 122.929012 121.870397) (xy 122.929012 121.127899) (xy 123.453646 121.127899)
 				)
 			)
 			(polygon
 				(pts
-					(xy 124.593771 121.127899) (xy 123.851884 123.16) (xy 123.26448 123.16) (xy 122.522592 121.127899)
-					(xy 123.073115 121.127899) (xy 123.56502 122.555376) (xy 124.056803 121.127899)
-				)
-			)
-			(polygon
-				(pts
-					(xy 125.806437 123.199078) (xy 125.656398 123.191372) (xy 125.517241 123.168886) (xy 125.387683 123.132278)
-					(xy 125.264342 123.079711) (xy 125.154835 123.013392) (xy 125.057711 122.933098) (xy 124.97379 122.839121)
-					(xy 124.902533 122.72972) (xy 124.843876 122.603004) (xy 124.802854 122.469048) (xy 124.77707 122.317581)
-					(xy 124.768039 122.146025) (xy 124.776489 121.986333) (xy 124.800952 121.840977) (xy 124.840457 121.70822)
-					(xy 124.89675 121.582069) (xy 124.966806 121.470203) (xy 125.050872 121.371165) (xy 125.14474 121.289083)
-					(xy 125.25363 121.21953) (xy 125.379378 121.162459) (xy 125.51197 121.122064) (xy 125.654297 121.0973)
-					(xy 125.80778 121.08882) (xy 125.933124 121.092626) (xy 126.039323 121.10323) (xy 126.229954 121.140844)
-					(xy 126.395917 121.199096) (xy 126.526465 121.258691) (xy 126.526465 121.753161) (xy 126.466381 121.753161)
-					(xy 126.369905 121.674392) (xy 126.238136 121.584633) (xy 126.160544 121.544149) (xy 126.075593 121.510017)
-					(xy 125.985922 121.48735) (xy 125.888381 121.479609) (xy 125.779871 121.488407) (xy 125.677965 121.514413)
-					(xy 125.58312 121.559954) (xy 125.493562 121.629818) (xy 125.422341 121.717585) (xy 125.363014 121.836081)
-					(xy 125.32658 121.972359) (xy 125.313189 122.147369) (xy 125.319882 122.274203) (xy 125.338472 122.379631)
-					(xy 125.367166 122.46696) (xy 125.430166 122.584629) (xy 125.503087 122.668949) (xy 125.591761 122.733596)
-					(xy 125.688956 122.776172) (xy 125.791647 122.800403) (xy 125.891189 122.80829) (xy 125.986013 122.801036)
-					(xy 126.080355 122.779103) (xy 126.170796 122.744511) (xy 126.253157 122.699968) (xy 126.377477 122.613872)
-					(xy 126.471755 122.534738) (xy 126.526465 122.534738) (xy 126.526465 123.023346) (xy 126.380163 123.087948)
-					(xy 126.234106 123.140094) (xy 126.046894 123.183935) (xy 125.951259 123.194753)
+					(xy 125.566102 121.518688) (xy 124.930826 121.518688) (xy 124.930826 123.16) (xy 124.406193 123.16)
+					(xy 124.406193 121.518688) (xy 123.770917 121.518688) (xy 123.770917 121.127899) (xy 125.566102 121.127899)
 				)
 			)
