File: hardware/kicad/scoopy/scoopy.kicad_sch (KiCad schematic)
At the start: 11 parts, among them J1 ESP32_SuperMini, J2 LD2410C, J3 Conn_01x04_Pin, SW1 SW_Push, SW2 SW_Push

Commit message: More schem info on kicad
Parts:
- D1: MPN MP008277 -> C22371297
- D2: MPN MP008288 -> C22371297
- D3: MPN MP008288 -> C19171390
- R1, R2, R3: MPN CR0603-FX-1001ELF -> C2907002
- SW1, SW2: MPN TL3305CF260QG -> C879462
Other:
- note added: "3v3 gnd Yellow to RX2. Green to TX2."
Changed lines of the file:
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@@
+		)
+	)
+	(text "3v3 gnd\nYellow to RX2. Green to TX2. "
+		(exclude_from_sim no)
+		(at 60.706 94.996 0)
+		(effects
+			(font
+				(size 1.27 1.27)
+			)
 		)
 	)
@@
 			)
 		)
-		(property "MPN" "TL3305CF260QG"
+		(property "MPN" "C879462"
 			(at 101.6 33.02 0)
 			(hide yes)
@@
 			)
 		)
-		(property "MPN" "TL3305CF260QG"
+		(property "MPN" "C879462"
 			(at 101.6 27.94 0)
 			(hide yes)
@@
 			)
 		)
-		(property "MPN" "MP008288"
+		(property "MPN" "C19171390"
 			(at 111.76 59.69 0)
 			(hide yes)
@@
 			)
 		)
-		(property "MPN" "MP008288"
+		(property "MPN" "C22371297"
 			(at 111.76 53.34 0)
 			(hide yes)
@@
 			)
 		)
-		(property "MPN" "CR0603-FX-1001ELF"
+		(property "MPN" "C2907002"
 			(at 100.33 59.69 90)
 			(hide yes)
@@
 			)
 		)
-		(property "MPN" "MP008277"
+		(property "MPN" "C22371297"
 			(at 111.76 44.45 0)
 			(hide yes)
@@
 			)
 		)
-		(property "MPN" "CR0603-FX-1001ELF"
+		(property "MPN" "C2907002"
 			(at 100.33 44.45 90)
 			(hide yes)
@@
 			)
 		)
-		(property "MPN" "CR0603-FX-1001ELF"
+		(property "MPN" "C2907002"
 			(at 100.33 53.34 90)
 			(hide yes)

Commit message: 1k Res was too bright for LEDs. Changed to 2.2k
Parts:
- R1, R2, R3: value 1k -> 2.2k; Link https://uk.farnell.com/bourns/cr0603-fx-1001elf/res-1k-1-0-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 -> https://uk.farnell.com/multicomp-pro/mcwr06x2201ftl/res-2k2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; Supplier_PN 2008335 -> MCWR06X2201FTL
Other:
- note removed: "3v3 gnd Yellow to RX2. Green to TX2."
Changed lines of the file:
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@@
-		)
-	)
-	(text "3v3 gnd\nYellow to RX2. Green to TX2. "
-		(exclude_from_sim no)
-		(at 60.706 94.996 0)
-		(effects
-			(font
-				(size 1.27 1.27)
-			)
 		)
 	)
@@
 			)
 		)
-		(property "Value" "1k"
+		(property "Value" "2.2k"
 			(at 99.568 55.372 90)
 			(show_name no)
@@
 			)
 		)
-		(property "Datasheet" "https://www.farnell.com/datasheets/3693949.pdf"
+		(property "Datasheet" "https://4donline.ihs.com/images/VipMasterIC/IC/SCMP/SCMP-S-A0009547702/SCMP-S-A0009547702-1.pdf?hkey=6D3A4C79FDBF58556ACFDE234799DDF0"
 			(at 100.33 59.69 0)
 			(hide yes)
@@
 			)
 		)
-		(property "Supplier_PN" "2008335"
+		(property "Supplier_PN" "MCWR06X2201FTL"
 			(at 100.33 59.69 90)
 			(hide yes)
@@
 			)
 		)
-		(property "Link" "https://uk.farnell.com/bourns/cr0603-fx-1001elf/res-1k-1-0-1w-0603-thick-film/dp/2008335"
+		(property "Link" "https://uk.farnell.com/multicomp-pro/mcwr06x2201ftl/res-2k2-1-0-1w-0603-thick-film/dp/2447320"
 			(at 100.33 59.69 90)
 			(hide yes)
@@
 			)
 		)
-		(property "Value" "1k"
+		(property "Value" "2.2k"
 			(at 99.822 40.132 90)
 			(show_name no)
@@
 			)
 		)
-		(property "Datasheet" "https://www.farnell.com/datasheets/3693949.pdf"
+		(property "Datasheet" "https://4donline.ihs.com/images/VipMasterIC/IC/SCMP/SCMP-S-A0009547702/SCMP-S-A0009547702-1.pdf?hkey=6D3A4C79FDBF58556ACFDE234799DDF0"
 			(at 100.33 44.45 0)
 			(hide yes)
@@
 			)
 		)
-		(property "Supplier_PN" "2008335"
+		(property "Supplier_PN" "MCWR06X2201FTL"
 			(at 100.33 44.45 90)
 			(hide yes)
@@
 			)
 		)
-		(property "Link" "https://uk.farnell.com/bourns/cr0603-fx-1001elf/res-1k-1-0-1w-0603-thick-film/dp/2008335"
+		(property "Link" "https://uk.farnell.com/multicomp-pro/mcwr06x2201ftl/res-2k2-1-0-1w-0603-thick-film/dp/2447320"
 			(at 100.33 44.45 90)
 			(hide yes)
@@
 			)
 		)
-		(property "Value" "1k"
+		(property "Value" "2.2k"
 			(at 99.568 49.022 90)
 			(show_name no)
@@
 			)
 		)
-		(property "Datasheet" "https://www.farnell.com/datasheets/3693949.pdf"
+		(property "Datasheet" "https://4donline.ihs.com/images/VipMasterIC/IC/SCMP/SCMP-S-A0009547702/SCMP-S-A0009547702-1.pdf?hkey=6D3A4C79FDBF58556ACFDE234799DDF0"
 			(at 100.33 53.34 0)
 			(hide yes)
@@
 			)
 		)
-		(property "Supplier_PN" "2008335"
+		(property "Supplier_PN" "MCWR06X2201FTL"
 			(at 100.33 53.34 90)
 			(hide yes)
@@
 			)
 		)
-		(property "Link" "https://uk.farnell.com/bourns/cr0603-fx-1001elf/res-1k-1-0-1w-0603-thick-film/dp/2008335"
+		(property "Link" "https://uk.farnell.com/multicomp-pro/mcwr06x2201ftl/res-2k2-1-0-1w-0603-thick-film/dp/2447320"
 			(at 100.33 53.34 90)
 			(hide yes)

Commit message: Updated proper ESP32-C3 supermini in eBOM
Parts:
- J2: MPN (none) -> C19723500
- R1, R2, R3: MPN C2907002 -> C2907005
Changed lines of the file:
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@@
+			)
+		)
+		(property "MPN" "C19723500"
+			(at 19.05 93.98 0)
+			(hide yes)
+			(show_name no)
+			(do_not_autoplace no)
+			(effects
+				(font
+					(size 1.27 1.27)
+				)
 			)
 		)
@@
 			)
 		)
-		(property "MPN" "C2907002"
+		(property "MPN" "C2907005"
 			(at 100.33 59.69 90)
 			(hide yes)
@@
 			)
 		)
-		(property "MPN" "C2907002"
+		(property "MPN" "C2907005"
 			(at 100.33 44.45 90)
 			(hide yes)
@@
 			)
 		)
-		(property "MPN" "C2907002"
+		(property "MPN" "C2907005"
 			(at 100.33 53.34 90)
 			(hide yes)
